File: hardware/hexasense.brd (EAGLE design)
At the start: 100 x 62 mm, 41 parts

Commit message: more routing...
Routing:
- net N$4: track 0.00 -> 91.8 mm, vias 0 -> 3
- net N$7: track 0.00 -> 78.1 mm, vias 0 -> 1
- net N$19: track 0.00 -> 75.8 mm, vias 0 -> 1
- net +3V3: track 279.4 -> 309.0 mm, vias 2 -> 3
- net DATA: track 48.7 -> 68.2 mm
- net GND: track 40.5 -> 57.2 mm, vias 2 -> 3
Changed lines of the file:
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@@
 <wire x1="24.95" y1="48.77" x2="24.96" y2="48.76" width="0.254" layer="16"/>
 <wire x1="24.96" y1="48.76" x2="24.96" y2="51.3" width="0.254" layer="1"/>
-<wire x1="41.11" y1="43.83" x2="41.1" y2="46.905" width="0" layer="19" extent="16-16"/>
-<wire x1="41.11" y1="41.29" x2="41.11" y2="43.83" width="0" layer="19" extent="1-1"/>
-<wire x1="45" y1="28.75" x2="41.11" y2="41.29" width="0" layer="19" extent="1-1"/>
-<wire x1="68.8" y1="6.555" x2="68.8" y2="17.985" width="0" layer="19" extent="1-1"/>
-<wire x1="15" y1="28.75" x2="28.05" y2="25.995" width="0" layer="19" extent="1-1"/>
 <wire x1="24.96" y1="48.76" x2="27.07" y2="48.76" width="0.254" layer="16"/>
 <wire x1="27.07" y1="48.76" x2="28.65" y2="50.34" width="0.254" layer="16"/>
@@
 <wire x1="37.41" y1="46.89" x2="41.085" y2="46.89" width="0.254" layer="16"/>
 <wire x1="41.085" y1="46.89" x2="41.1" y2="46.905" width="0.254" layer="16"/>
+<via x="16.32" y="26.71" extent="1-16" drill="0.3"/>
+<wire x1="41.11" y1="41.29" x2="41.11" y2="43.83" width="0.254" layer="16"/>
+<wire x1="41.11" y1="41.29" x2="43.51" y2="38.89" width="0.254" layer="1"/>
+<wire x1="43.51" y1="38.89" x2="43.51" y2="30.24" width="0.254" layer="1"/>
+<wire x1="43.51" y1="30.24" x2="45" y2="28.75" width="0.254" layer="1"/>
+<wire x1="41.11" y1="43.83" x2="41.085" y2="46.89" width="0" layer="19" extent="16-16"/>
+<wire x1="68.8" y1="17.985" x2="45" y2="28.75" width="0" layer="19" extent="1-1"/>
+<wire x1="68.8" y1="6.555" x2="68.8" y2="17.985" width="0" layer="19" extent="1-1"/>
 </signal>
 <signal name="+3V3">
@@
 <wire x1="33.5" y1="18.89" x2="37.57" y2="18.89" width="0.254" layer="1"/>
 <wire x1="37.57" y1="18.89" x2="37.97" y2="18.49" width="0.254" layer="1"/>
-<wire x1="41.11" y1="36.21" x2="41.1" y2="48.175" width="0" layer="19" extent="16-16"/>
-<wire x1="59.6" y1="4.015" x2="50.07" y2="11.06" width="0" layer="19" extent="1-1"/>
-<wire x1="24.96" y1="43.68" x2="41.1" y2="48.175" width="0" layer="19" extent="16-16"/>
+<wire x1="24.96" y1="43.68" x2="32.67" y2="43.68" width="0.254" layer="1"/>
+<wire x1="32.67" y1="43.68" x2="32.83" y2="43.68" width="0.254" layer="1"/>
+<wire x1="32.83" y1="43.68" x2="37.33" y2="48.18" width="0.254" layer="1"/>
+<via x="37.33" y="48.18" extent="1-16" drill="0.3"/>
+<wire x1="37.33" y1="48.18" x2="41.095" y2="48.18" width="0.254" layer="16"/>
+<wire x1="41.095" y1="48.18" x2="41.1" y2="48.175" width="0.254" layer="16"/>
+<wire x1="41.11" y1="36.21" x2="40.14" y2="36.21" width="0.254" layer="1"/>
+<wire x1="40.14" y1="36.21" x2="32.67" y2="43.68" width="0.254" layer="1"/>
+<wire x1="50.07" y1="11.06" x2="59.6" y2="4.015" width="0" layer="19" extent="1-1"/>
 </signal>
 <signal name="TEMP_1">
@@
 <wire x1="17.66" y1="44.73" x2="19.15" y2="46.22" width="0.254" layer="16"/>
 <wire x1="19.15" y1="46.22" x2="24.96" y2="46.22" width="0.254" layer="16"/>
-<wire x1="24.96" y1="46.22" x2="41.11" y2="38.75" width="0" layer="19" extent="1-1"/>
+<wire x1="41.11" y1="38.75" x2="41.11" y2="39.28" width="0.254" layer="16"/>
+<wire x1="41.11" y1="39.28" x2="35.47" y2="44.92" width="0.254" layer="16"/>
+<wire x1="35.47" y1="44.92" x2="26.26" y2="44.92" width="0.254" layer="16"/>
+<wire x1="26.26" y1="44.92" x2="24.96" y2="46.22" width="0.254" layer="16"/>
 </signal>
 <signal name="SDA">
@@
 <contactref element="LED4" pad="K"/>
 <contactref element="U$3" pad="P$7"/>
-<wire x1="14.1" y1="60.27" x2="68.8" y2="11.635" width="0" layer="19" extent="1-1"/>
+<wire x1="14.1" y1="60.27" x2="19.2" y2="60.27" width="0.254" layer="16"/>
+<wire x1="19.2" y1="60.27" x2="20.53" y2="58.94" width="0.254" layer="16"/>
+<wire x1="20.53" y1="58.94" x2="36.98" y2="58.94" width="0.254" layer="16"/>
+<wire x1="36.98" y1="58.94" x2="56.39" y2="39.53" width="0.254" layer="16"/>
+<wire x1="56.39" y1="39.53" x2="63.72" y2="39.53" width="0.254" layer="16"/>
+<via x="63.72" y="39.53" extent="1-16" drill="0.3"/>
+<wire x1="63.72" y1="39.53" x2="63.72" y2="17.02" width="0.254" layer="1"/>
+<wire x1="63.72" y1="17.02" x2="64.67" y2="16.07" width="0.254" layer="1"/>
+<wire x1="64.67" y1="16.07" x2="64.67" y2="15.19" width="0.254" layer="1"/>
+<wire x1="64.67" y1="15.19" x2="63.03" y2="13.55" width="0.254" layer="1"/>
+<via x="63.03" y="13.55" extent="1-16" drill="0.3"/>
+<wire x1="63.03" y1="13.55" x2="64.95" y2="11.63" width="0.254" layer="16"/>
+<wire x1="64.95" y1="11.63" x2="65.85" y2="11.63" width="0.254" layer="16"/>
+<via x="65.85" y="11.63" extent="1-16" drill="0.3"/>
+<wire x1="65.85" y1="11.63" x2="65.855" y2="11.635" width="0.254" layer="1"/>
+<wire x1="65.855" y1="11.635" x2="68.8" y2="11.635" width="0.254" layer="1"/>
 </signal>
 <signal name="N$5">
@@
 <contactref element="LED7" pad="K"/>
 <contactref element="U$3" pad="P$10"/>
-<wire x1="18.87" y1="53" x2="68.8" y2="15.445" width="0" layer="19" extent="1-1"/>
+<wire x1="18.87" y1="53" x2="42.03" y2="53" width="0.254" layer="16"/>
+<wire x1="42.03" y1="53" x2="56.16" y2="38.87" width="0.254" layer="16"/>
+<wire x1="56.16" y1="38.87" x2="64.97" y2="38.87" width="0.254" layer="16"/>
+<via x="64.97" y="38.87" extent="1-16" drill="0.3"/>
+<wire x1="64.97" y1="38.87" x2="64.97" y2="17.38" width="0.254" layer="1"/>
+<wire x1="64.97" y1="17.38" x2="66.91" y2="15.44" width="0.254" layer="1"/>
+<wire x1="66.91" y1="15.44" x2="68.795" y2="15.44" width="0.254" layer="1"/>
+<wire x1="68.795" y1="15.44" x2="68.8" y2="15.445" width="0.254" layer="1"/>
 </signal>
 <signal name="N$8">
@@
 <contactref element="LED10" pad="K"/>
 <contactref element="U$3" pad="P$14"/>
-<wire x1="59.6" y1="16.715" x2="21.1" y2="60.27" width="0" layer="19" extent="1-1"/>
+<via x="62.5" y="40.35" extent="1-16" drill="0.3"/>
+<wire x1="62.5" y1="17.34" x2="61.88" y2="16.72" width="0.254" layer="1"/>
+<wire x1="61.88" y1="16.72" x2="59.605" y2="16.72" width="0.254" layer="1"/>
+<wire x1="59.605" y1="16.72" x2="59.6" y2="16.715" width="0.254" layer="1"/>
+<wire x1="21.1" y1="60.27" x2="42.58" y2="60.27" width="0.254" layer="16"/>
+<wire x1="42.58" y1="60.27" x2="62.5" y2="40.35" width="0.254" layer="16"/>
+<wire x1="62.5" y1="17.34" x2="62.5" y2="40.35" width="0.254" layer="1"/>
 </signal>
 <signal name="N$20">

Commit message: more routing...
Routing:
- net S1: track 0.00 -> 84.4 mm, vias 0 -> 1
- net S2: track 0.00 -> 74.5 mm, vias 0 -> 6
- net N$2: track 0.00 -> 68.2 mm, vias 0 -> 1
- net N$9: track 0.00 -> 53.9 mm, vias 0 -> 2
- net +5V: track 103.2 -> 153.6 mm, vias 0 -> 3
- net N$8: track 0.00 -> 41.7 mm, vias 0 -> 2
- net SDA: track 152.6 -> 153.3 mm
- net GND: vias 3 -> 4

Commit message: finished routing
Routing:
- net SCL: track 117.1 -> 144.0 mm, vias 0 -> 3
- net +3V3: track 309.0 -> 333.8 mm, vias 3 -> 5
- net SDA: track 153.3 -> 172.9 mm, vias 1 -> 3
- net TEMP_2: track 48.3 -> 53.2 mm
- net TEMP_1: track 63.2 -> 63.9 mm
- net GND: vias 4 -> 7
Changed lines of the file:
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@@
 <wire x1="13.4" y1="10.25" x2="13.4" y2="26.25" width="2" layer="46"/>
 <wire x1="13.4" y1="26.25" x2="0" y2="26.25" width="2" layer="46"/>
-<text x="58.02" y="74.2" size="1.778" layer="1" font="vector" ratio="10" rot="SR270">HexaSense</text>
-<text x="53.29" y="73.37" size="1.778" layer="1" font="vector" ratio="10" rot="SR270">Display</text>
-<text x="50.22" y="73.6" size="1.778" layer="1" font="vector" ratio="10" rot="SR270">20130114</text>
+<text x="96.52" y="47.5" size="1.778" layer="1" font="vector" ratio="10" rot="SR270">HexaSense</text>
+<text x="96" y="29" size="1.778" layer="1" font="vector" ratio="10" rot="SR270">Display</text>
+<text x="52" y="57.93" size="1.778" layer="1" font="vector" ratio="10" rot="SR0">20130114</text>
 <hole x="96" y="58" drill="4"/>
 <hole x="96" y="4" drill="4"/>
@@
 <wire x1="43.51" y1="30.24" x2="45" y2="28.75" width="0.254" layer="1"/>
 <via x="70.53" y="18.27" extent="1-16" drill="0.3"/>
-<wire x1="90.79" y1="29.54" x2="91.095" y2="31.03" width="0" layer="19" extent="16-16"/>
-<wire x1="75" y1="28.75" x2="90.79" y2="29.54" width="0" layer="19" extent="1-1"/>
-<wire x1="70.53" y1="18.27" x2="75" y2="28.75" width="0" layer="19" extent="1-1"/>
-<wire x1="68.8" y1="17.985" x2="70.53" y2="18.27" width="0" layer="19" extent="1-1"/>
-<wire x1="68.8" y1="6.555" x2="68.8" y2="17.985" width="0" layer="19" extent="1-1"/>
-<wire x1="68.8" y1="5.285" x2="68.8" y2="6.555" width="0" layer="19" extent="1-1"/>
-<wire x1="68.8" y1="4.015" x2="68.8" y2="5.285" width="0" layer="19" extent="1-1"/>
-<wire x1="45" y1="28.75" x2="68.8" y2="17.985" width="0" layer="19" extent="1-1"/>
-<wire x1="41.085" y1="46.89" x2="41.11" y2="43.83" width="0" layer="19" extent="16-16"/>
-<wire x1="42.72" y1="25.99" x2="45" y2="28.75" width="0" layer="19" extent="1-1"/>
-<wire x1="3.2" y1="49.27" x2="5.99" y2="46.895" width="0" layer="19" extent="16-16"/>
-<wire x1="3.2" y1="51.81" x2="3.2" y2="49.27" width="0" layer="19" extent="1-1"/>
-<wire x1="33.89" y1="22.695" x2="42.72" y2="25.99" width="0" layer="19" extent="1-1"/>
-<wire x1="33.89" y1="20.155" x2="33.89" y2="22.695" width="0" layer="19" extent="1-1"/>
-<wire x1="31.35" y1="18.885" x2="33.89" y2="20.155" width="0" layer="19" extent="1-1"/>
-<wire x1="33.89" y1="15.075" x2="31.35" y2="18.885" width="0" layer="19" extent="1-1"/>
-<wire x1="28.05" y1="25.995" x2="33.89" y2="22.695" width="0" layer="19" extent="1-1"/>
-<wire x1="28.05" y1="10.505" x2="33.89" y2="15.075" width="0" layer="19" extent="1-1"/>
-<wire x1="35.5" y1="7.55" x2="33.89" y2="15.075" width="0" layer="19" extent="1-1"/>
-<wire x1="37.97" y1="3.25" x2="35.5" y2="7.55" width="0" layer="19" extent="1-1"/>
-<wire x1="16.32" y1="26.71" x2="28.05" y2="25.995" width="0" layer="19" extent="1-1"/>
-<wire x1="15" y1="28.75" x2="16.32" y2="26.71" width="0" layer="19" extent="1-1"/>
+<via x="72.66" y="28.69" extent="1-16" drill="0.3"/>
+<via x="89.46" y="24.19" extent="1-16" drill="0.3"/>
+<via x="70.96" y="2.73" extent="1-16" drill="0.3"/>
+<wire x1="41.11" y1="43.83" x2="41.085" y2="46.89" width="0" layer="19" extent="16-16"/>
 </signal>
 <signal name="+3V3">
@@
 <contactref element="U$8" pad="VDD"/>
 <contactref element="U$7" pad="VDD"/>
-<wire x1="45.2" y1="15" x2="49.14" y2="11.06" width="0.254" layer="1"/>
+<wire x1="45.2" y1="15" x2="49.08" y2="11.12" width="0.254" layer="1"/>
 <wire x1="49.14" y1="11.06" x2="50.07" y2="11.06" width="0.254" layer="1"/>
 <wire x1="45.2" y1="15" x2="38.78" y2="15" width="0.254" layer="1"/>
@@
 <wire x1="41.11" y1="36.21" x2="40.14" y2="36.21" width="0.254" layer="1"/>
 <wire x1="40.14" y1="36.21" x2="32.67" y2="43.68" width="0.254" layer="1"/>
-<wire x1="50.07" y1="11.06" x2="59.6" y2="4.015" width="0" layer="19" extent="1-1"/>
+<wire x1="59.6" y1="4.015" x2="51.345" y2="4.015" width="0.254" layer="1"/>
+<wire x1="51.345" y1="4.015" x2="48.97" y2="1.64" width="0.254" layer="1"/>
+<wire x1="48.97" y1="1.64" x2="47.6" y2="1.64" width="0.254" layer="1"/>
+<wire x1="47.6" y1="1.64" x2="46.71" y2="2.53" width="0.254" layer="1"/>
+<wire x1="46.71" y1="2.53" x2="46.71" y2="8.19" width="0.254" layer="1"/>
+<via x="46.71" y="8.19" extent="1-16" drill="0.3"/>
+<wire x1="46.71" y1="8.19" x2="46.71" y2="10.55" width="0.254" layer="16"/>
+<wire x1="46.71" y1="10.55" x2="47.28" y2="11.12" width="0.254" layer="16"/>
+<via x="47.28" y="11.12" extent="1-16" drill="0.3"/>
+<wire x1="47.28" y1="11.12" x2="49.08" y2="11.12" width="0.254" layer="1"/>
+<wire x1="49.08" y1="11.12" x2="49.14" y2="11.06" width="0.254" layer="1"/>
 </signal>
 <signal name="TEMP_1">
@@
 <contactref element="U$4" pad="PA4"/>
 <wire x1="31.35" y1="16.345" x2="32.74" y2="14.955" width="0.254" layer="16"/>
-<wire x1="32.74" y1="14.955" x2="32.74" y2="13.08" width="0.254" layer="16"/>
-<wire x1="32.74" y1="13.08" x2="39.18" y2="6.64" width="0.254" layer="16"/>
-<wire x1="39.18" y1="6.64" x2="70.43" y2="6.64" width="0.254" layer="16"/>
-<wire x1="70.43" y1="6.64" x2="75.68" y2="1.39" width="0.254" layer="16"/>
+<wire x1="32.74" y1="14.955" x2="32.74" y2="11.97" width="0.254" layer="16"/>
+<wire x1="39.51" y1="5.2" x2="71.87" y2="5.2" width="0.254" layer="16"/>
 <wire x1="84.88" y1="1.39" x2="86.23" y2="2.74" width="0.254" layer="16"/>
 <wire x1="86.23" y1="2.74" x2="86.23" y2="3.25" width="0.254" layer="16"/>
 <wire x1="75.68" y1="1.39" x2="84.88" y2="1.39" width="0.254" layer="16"/>
+<wire x1="39.51" y1="5.2" x2="32.74" y2="11.97" width="0.254" layer="16"/>
+<wire x1="75.68" y1="1.39" x2="71.87" y2="5.2" width="0.254" layer="16"/>
 </signal>
 <signal name="DATA">
@@
 <wire x1="27.35" y1="47.62" x2="29.35" y2="45.62" width="0.254" layer="16"/>
 <wire x1="41.085" y1="45.62" x2="29.35" y2="45.62" width="0.254" layer="16"/>
-<wire x1="59.6" y1="5.285" x2="47.1" y2="15" width="0" layer="19" extent="1-1"/>
 <wire x1="64.46" y1="10.77" x2="64.12" y2="10.43" width="0.254" layer="16"/>
+<wire x1="59.6" y1="5.285" x2="51.665" y2="5.285" width="0.254" layer="1"/>
+<wire x1="51.665" y1="5.285" x2="50.11" y2="6.84" width="0.254" layer="1"/>
+<via x="50.11" y="6.84" extent="1-16" drill="0.3"/>
+<wire x1="50.11" y1="6.84" x2="50.11" y2="11.61" width="0.254" layer="16"/>
+<wire x1="50.11" y1="11.61" x2="48.85" y2="12.87" width="0.254" layer="16"/>
+<via x="48.85" y="12.87" extent="1-16" drill="0.3"/>
+<wire x1="48.85" y1="12.87" x2="47.1" y2="14.62" width="0.254" layer="1"/>
+<wire x1="47.1" y1="14.62" x2="47.1" y2="15" width="0.254" layer="1"/>
 </signal>
 <signal name="SCL">
@@
 <wire x1="41.1" y1="49.445" x2="44.485" y2="49.475" width="0.254" layer="16"/>
 <wire x1="85.365" y1="34.22" x2="88.555" y2="31.03" width="0.254" layer="16"/>
-<wire x1="44.485" y1="49.475" x2="55.77" y2="38.19" width="0.254" layer="16"/>
-<wire x1="55.77" y1="38.19" x2="68" y2="38.19" width="0.254" layer="16"/>
+<wire x1="44.485" y1="49.475" x2="55.81" y2="38.15" width="0.254" layer="16"/>
 <wire x1="68" y1="38.19" x2="71.97" y2="34.22" width="0.254" layer="16"/>
 <wire x1="71.97" y1="34.22" x2="85.365" y2="34.22" width="0.254" layer="16"/>
@@
 <wire x1="51.22" y1="20.43" x2="51.91" y2="19.74" width="0.254" layer="1"/>
 <wire x1="51.91" y1="19.74" x2="51.91" y2="14.91" width="0.254" layer="1"/>
-<wire x1="55.77" y1="38.19" x2="51.22" y2="20.43" width="0" layer="19" extent="1-16"/>
+<wire x1="51.22" y1="20.43" x2="58.38" y2="20.43" width="0.254" layer="1"/>
+<via x="58.38" y="20.43" extent="1-16" drill="0.3"/>
+<wire x1="58.38" y1="20.43" x2="60.18" y2="22.23" width="0.254" layer="16"/>
+<wire x1="60.18" y1="22.23" x2="60.18" y2="34.84" width="0.254" layer="16"/>
+<via x="60.18" y="34.84" extent="1-16" drill="0.3"/>
+<wire x1="55.81" y1="38.15" x2="57.11" y2="38.15" width="0.254" layer="16"/>
+<via x="57.11" y="38.15" extent="1-16" drill="0.3"/>
+<wire x1="57.11" y1="38.15" x2="60.18" y2="35.08" width="0.254" layer="1"/>
+<wire x1="60.18" y1="35.08" x2="60.18" y2="34.84" width="0.254" layer="1"/>
+<wire x1="68" y1="38.19" x2="57.15" y2="38.19" width="0.254" layer="16"/>
+<wire x1="57.15" y1="38.19" x2="57.11" y2="38.15" width="0.254" layer="16"/>
 </signal>
 <signal name="BTN">
@@
 <contactref element="S3" pad="1"/>
 <contactref element="U$4" pad="PA3"/>
-<wire x1="84.95" y1="23.3" x2="84.932940625" y2="18.960028125" width="0" layer="19" extent="1-16"/>
 <via x="84.9" y="10.58" extent="1-16" drill="0.3"/>
 <wire x1="84.932940625" y1="18.960028125" x2="84.9" y2="10.58" width="0.254" layer="1"/>
@@
 <contactref element="U$4" pad="PA0"/>
 <contactref element="U$1" pad="4"/>
+<wire x1="70.8" y1="8.52" x2="57.89" y2="8.52" width="0.254" layer="16"/>
+<wire x1="57.89" y1="8.52" x2="55.12" y2="6.04" width="0.254" layer="16"/>
+<wire x1="55.12" y1="6.04" x2="40.215" y2="6.04" width="0.254" layer="16"/>
+<wire x1="40.215" y1="6.04" x2="37" y2="9.255" width="0.254" layer="16"/>
+<wire x1="37" y1="9.255" x2="37" y2="14.505" width="0.254" layer="16"/>
+<wire x1="37" y1="14.505" x2="33.89" y2="17.615" width="0.254" layer="16"/>
 <wire x1="76.07" y1="3.25" x2="70.8" y2="8.52" width="0.254" layer="16"/>
-<wire x1="70.8" y1="8.52" x2="42.73" y2="8.52" width="0.254" layer="16"/>
-<wire x1="42.73" y1="8.52" x2="33.89" y2="17.36" width="0.254" layer="16"/>
-<wire x1="33.89" y1="17.36" x2="33.89" y2="17.615" width="0.254" layer="16"/>
 </signal>
 <signal name="N$19">

Commit message: passing the DRC
Routing:
- net S3: track 34.6 -> 0.00 mm, vias 1 -> 0
- net +5V: track 153.6 -> 150.3 mm
- net +3V3: track 333.8 -> 336.2 mm
- net S1: track 84.4 -> 85.4 mm
- net SCL: track 144.0 -> 143.7 mm, vias 3 -> 1
