File: hardware/power.brd (EAGLE design)
At the start: 50 x 50 mm, 36 parts, among them U1 LM324D, U2 LM324D, U3 LM1117MP-3.3

Commit message: fixed wrong wiring at voltage regulator
Connections:
- removed net N$15: C1.1, U3.1
- net +5V: now also C1.1
- net GND: now also U3.1
Routing:
- net +5V: track 47.7 -> 65.7 mm
- net N$15: track 3.62 -> 0.00 mm
Other:
- board text added: "20130806"
- board text removed: "20130207"
Changed lines of the file:
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@@
 <wire x1="-6" y1="-6" x2="-6" y2="56" width="0" layer="48" style="longdash"/>
 <wire x1="-6" y1="56" x2="54" y2="56" width="0" layer="48" style="longdash"/>
-<text x="49.1" y="44.95" size="1.016" layer="1" font="vector" ratio="15" rot="R180">20130207</text>
+<text x="49.1" y="44.95" size="1.016" layer="1" font="vector" ratio="15" rot="R180">20130806</text>
 <text x="49.1" y="49.1" size="1.27" layer="1" font="vector" ratio="15" rot="R180">Hexasense
 Power</text>
@@
 <via x="22.3" y="11.15" extent="1-16" drill="0.3"/>
 <via x="26.95" y="35" extent="1-16" drill="0.3"/>
+<contactref element="U3" pad="1"/>
 </signal>
 <signal name="N$11">
@@
 <wire x1="18.7" y1="7.35" x2="32.85" y2="7.35" width="0.254" layer="16"/>
 <wire x1="32.85" y1="7.35" x2="40" y2="14.5" width="0.254" layer="16"/>
-</signal>
-<signal name="N$15">
-<contactref element="U3" pad="1"/>
 <contactref element="C1" pad="1"/>
-<wire x1="33.95" y1="3" x2="36.2004" y2="5.2504" width="0.254" layer="1"/>
-<wire x1="36.2004" y1="5.2504" x2="36.2004" y2="5.6886" width="0.254" layer="1"/>
+<wire x1="33.95" y1="3" x2="38.9" y2="3" width="0.254" layer="1"/>
+<wire x1="38.9" y1="3" x2="41.4" y2="5.5" width="0.254" layer="1"/>
+<wire x1="41.4" y1="5.5" x2="41.4" y2="13.1" width="0.254" layer="1"/>
+<wire x1="41.4" y1="13.1" x2="40" y2="14.5" width="0.254" layer="1"/>
 </signal>
 </signals>

Commit message: changed testpoints to SMD pads
Parts:
- GND, OFFSET-1, OFFSET-2, PT100-1, PT100-2, TEMP-1, TEMP-2, U_M-1, U_M-2, VCC: value TPPAD1-13 -> TPB1,27; device testpad:P1-13 -> testpad:B1,27
Routing:
- net U_M_2: track 19.3 -> 20.0 mm, vias 2 -> 3
Other:
- board text added: "20130829"
- board text removed: "20130806"
Changed lines of the file:
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@@
 <wire x1="-6" y1="-6" x2="-6" y2="56" width="0" layer="48" style="longdash"/>
 <wire x1="-6" y1="56" x2="54" y2="56" width="0" layer="48" style="longdash"/>
-<text x="49.1" y="44.95" size="1.016" layer="1" font="vector" ratio="15" rot="R180">20130806</text>
+<text x="49.1" y="44.95" size="1.016" layer="1" font="vector" ratio="15" rot="R180">20130829</text>
 <text x="49.1" y="49.1" size="1.27" layer="1" font="vector" ratio="15" rot="R180">Hexasense
 Power</text>
@@
 </element>
 <element name="U$1" library="Reichelt" package="RJ45-REICHELT" value="MEBP8-8G" x="4.7" y="25" rot="R270"/>
-<element name="U_M-1" library="testpad" package="P1-13" value="TPPAD1-13" x="35.56" y="40.64" smashed="yes" rot="MR0">
+<element name="U_M-1" library="testpad" package="B1,27" value="TPB1,27" x="35.56" y="40.64" smashed="yes" rot="MR0">
 <attribute name="TP_SIGNAL_NAME" value="" x="36.195" y="38.735" size="1" layer="38" rot="MR0"/>
 <attribute name="NAME" x="34.395" y="40.156" size="1.27" layer="26" ratio="10" rot="MR0"/>
 <attribute name="VALUE" x="36.195" y="39.878" size="0.0254" layer="28" rot="MR0"/>
 </element>
-<element name="TEMP-1" library="testpad" package="P1-13" value="TPPAD1-13" x="17.78" y="27.94" rot="MR0">
+<element name="TEMP-1" library="testpad" package="B1,27" value="TPB1,27" x="17.78" y="27.94" rot="MR0">
 <attribute name="TP_SIGNAL_NAME" value="" x="17.78" y="27.94" size="1.778" layer="28" rot="MR0" display="off"/>
 </element>
-<element name="GND" library="testpad" package="P1-13" value="TPPAD1-13" x="17.78" y="45.72" rot="MR0">
+<element name="GND" library="testpad" package="B1,27" value="TPB1,27" x="17.78" y="45.72" rot="MR0">
 <attribute name="TP_SIGNAL_NAME" value="" x="17.78" y="45.72" size="1.778" layer="28" rot="MR0" display="off"/>
 </element>
-<element name="VCC" library="testpad" package="P1-13" value="TPPAD1-13" x="5.08" y="35.56" smashed="yes" rot="MR270">
+<element name="VCC" library="testpad" package="B1,27" value="TPB1,27" x="5.08" y="35.56" smashed="yes" rot="MR270">
 <attribute name="TP_SIGNAL_NAME" value="" x="6.985" y="36.195" size="1" layer="38" rot="MR270"/>
 <attribute name="NAME" x="2.205" y="34.164" size="1.27" layer="26" ratio="10" rot="MR180"/>
@@
 <attribute name="NAME" x="2.96" y="1.91" size="1.27" layer="25" rot="R90"/>
 </element>
-<element name="U_M-2" library="testpad" package="P1-13" value="TPPAD1-13" x="33.02" y="15.24" smashed="yes" rot="MR0">
+<element name="U_M-2" library="testpad" package="B1,27" value="TPB1,27" x="33.02" y="15.24" smashed="yes" rot="MR0">
 <attribute name="TP_SIGNAL_NAME" value="" x="33.655" y="13.335" size="1" layer="38" rot="MR0"/>
 <attribute name="NAME" x="35.505" y="17.206" size="1.27" layer="26" ratio="10" rot="MR0"/>
 <attribute name="VALUE" x="33.655" y="14.478" size="0.0254" layer="28" rot="MR0"/>
 </element>
-<element name="TEMP-2" library="testpad" package="P1-13" value="TPPAD1-13" x="17.78" y="22.86" smashed="yes" rot="MR0">
+<element name="TEMP-2" library="testpad" package="B1,27" value="TPB1,27" x="17.78" y="22.86" smashed="yes" rot="MR0">
 <attribute name="TP_SIGNAL_NAME" value="" x="18.415" y="20.955" size="1" layer="38" rot="MR0"/>
 <attribute name="NAME" x="22.265" y="20.526" size="1.27" layer="26" ratio="10" rot="MR0"/>
@@
 <attribute name="NAME" x="34.27" y="1.73" size="1.27" layer="25" rot="R180"/>
 </element>
-<element name="OFFSET-1" library="testpad" package="P1-13" value="TPPAD1-13" x="10.16" y="35.56" smashed="yes" rot="MR0">
+<element name="OFFSET-1" library="testpad" package="B1,27" value="TPB1,27" x="10.16" y="35.56" smashed="yes" rot="MR0">
 <attribute name="TP_SIGNAL_NAME" value="" x="10.795" y="33.655" size="1" layer="38" rot="MR0"/>
 <attribute name="NAME" x="6.865" y="38.474" size="1.27" layer="26" ratio="10" rot="MR180"/>
 <attribute name="VALUE" x="10.795" y="34.798" size="0.0254" layer="28" rot="MR0"/>
 </element>
-<element name="OFFSET-2" library="testpad" package="P1-13" value="TPPAD1-13" x="7.62" y="2.54" smashed="yes" rot="MR0">
+<element name="OFFSET-2" library="testpad" package="B1,27" value="TPB1,27" x="7.62" y="2.54" smashed="yes" rot="MR0">
 <attribute name="TP_SIGNAL_NAME" value="" x="8.255" y="0.635" size="1" layer="38" rot="MR0"/>
 <attribute name="NAME" x="17.755" y="1.706" size="1.27" layer="26" ratio="10" rot="MR0"/>
 <attribute name="VALUE" x="8.255" y="1.778" size="0.0254" layer="28" rot="MR0"/>
 </element>
-<element name="PT100-2" library="testpad" package="P1-13" value="TPPAD1-13" x="38.1" y="30.48" smashed="yes" rot="MR0">
+<element name="PT100-2" library="testpad" package="B1,27" value="TPB1,27" x="38.1" y="30.48" smashed="yes" rot="MR0">
 <attribute name="TP_SIGNAL_NAME" value="" x="38.735" y="28.575" size="1" layer="38" rot="MR0"/>
 <attribute name="NAME" x="37.435" y="29.896" size="1.27" layer="26" ratio="10" rot="MR0"/>
 <attribute name="VALUE" x="38.735" y="29.718" size="0.0254" layer="28" rot="MR0"/>
 </element>
-<element name="PT100-1" library="testpad" package="P1-13" value="TPPAD1-13" x="38.1" y="40.64" smashed="yes" rot="MR0">
+<element name="PT100-1" library="testpad" package="B1,27" value="TPB1,27" x="38.1" y="40.64" smashed="yes" rot="MR0">
 <attribute name="TP_SIGNAL_NAME" value="" x="38.735" y="38.735" size="1" layer="38" rot="MR0"/>
 <attribute name="NAME" x="39.165" y="41.474" size="1.27" layer="26" ratio="10" rot="MR180"/>
@@
 <wire x1="28.45" y1="8.05" x2="28.45" y2="9.65" width="0.254" layer="16"/>
 <wire x1="28.45" y1="9.65" x2="28.85" y2="10.05" width="0.254" layer="16"/>
-<wire x1="33.02" y1="15.24" x2="33.02" y2="14.22" width="0.254" layer="1"/>
-<wire x1="33.02" y1="14.22" x2="28.85" y2="10.05" width="0.254" layer="1"/>
+<wire x1="28.85" y1="10.05" x2="30" y2="10.05" width="0.254" layer="1"/>
+<wire x1="30" y1="10.05" x2="32.45" y2="12.5" width="0.254" layer="1"/>
+<via x="32.45" y="12.5" extent="1-16" drill="0.3"/>
+<wire x1="32.45" y1="12.5" x2="33.02" y2="13.07" width="0.254" layer="16"/>
+<wire x1="33.02" y1="13.07" x2="33.02" y2="15.24" width="0.254" layer="16"/>
 </signal>
 <signal name="U_M_1">
